File: Swadge-HW/Swadge-HW.kicad_sch (KiCad schematic)
At the start: 95 parts, among them J1 SAO, J2 PJ-307C, J3 PGM, P1 USB_C_Plug_USB2.0, Q1 Q_PMOS_GSD, SW1 YTS-D003-1A, SW2 YTS-D003-1A, SW3 YTS-D003-1A, SW4 YTS-D003-1A, SW5 YTS-D003-1A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

Commit message: Add electrolytic capacitor C26
add capacitor for noise management
Parts:
- added C26: 470μF, Swadge_Parts:C_Radial_D4_L5.4_P3.321, symbol Device:C_Polarized_US
Connections:
- net +3V3: now also C26.1
- net GND: now also C26.2
Changed lines of the file:
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@@
 	)
 	(junction
+		(at 166.37 189.23)
+		(diameter 0)
+		(color 0 0 0 0)
+	)
+	(junction
 		(at 328.93 113.03)
 		(diameter 0)
@@
 	)
 	(junction
+		(at 156.21 196.85)
+		(diameter 0)
+		(color 0 0 0 0)
+	)
+	(junction
 		(at 82.55 194.31)
 		(diameter 0)
@@
 	(wire
 		(pts
+			(xy 156.21 196.85) (xy 166.37 196.85)
+		)
+		(stroke
+			(width 0)
+			(type default)
+		)
+	)
+	(wire
+		(pts
 			(xy 134.62 173.99) (xy 134.62 176.53)
 		)
@@
 	(wire
 		(pts
-			(xy 156.21 189.23) (xy 160.02 189.23)
+			(xy 156.21 189.23) (xy 166.37 189.23)
 		)
 		(stroke
@@
 	(wire
 		(pts
+			(xy 166.37 189.23) (xy 170.18 189.23)
+		)
+		(stroke
+			(width 0)
+			(type default)
+		)
+	)
+	(wire
+		(pts
 			(xy 55.88 162.56) (xy 53.34 162.56)
 		)
@@
 	(symbol
 		(lib_id "Swadge_Parts:+3.3V")
-		(at 160.02 189.23 0)
+		(at 170.18 189.23 0)
 		(unit 1)
 		(exclude_from_sim no)
@@
 		(dnp no)
 		(property "Reference" "#PWR033"
-			(at 160.02 193.04 0)
+			(at 170.18 193.04 0)
 			(effects
 				(font
@@
 		)
 		(property "Value" "+3V3"
-			(at 162.814 189.23 0)
+			(at 165.862 187.198 0)
 			(effects
 				(font
@@
 		)
 		(property "Footprint" ""
-			(at 160.02 189.23 0)
+			(at 170.18 189.23 0)
 			(effects
 				(font
@@
 		)
 		(property "Datasheet" ""
-			(at 160.02 189.23 0)
+			(at 170.18 189.23 0)
 			(effects
 				(font
@@
 		)
 		(property "Description" ""
-			(at 160.02 189.23 0)
+			(at 170.18 189.23 0)
 			(effects
 				(font
@@
 		(exclude_from_sim no)
 		(in_bom yes)
-		(on_board no)
+		(on_board yes)
 		(dnp no)
 		(property "Reference" "D9"
@@
 					(unit 1)
 				)
+			)
+		)
+	)
+	(symbol
+		(lib_id "Device:C_Polarized_US")
+		(at 166.37 193.04 0)
+		(unit 1)
+		(exclude_from_sim no)
+		(in_bom yes)
+		(on_board yes)
+		(dnp no)
+		(property "Reference" "C26"
+			(at 167.005 190.5 0)
+			(effects
+				(font
+					(size 1.27 1.27)
+				)
+				(justify left)
+			)
+		)
+		(property "Value" "470μF"
+			(at 166.37 195.58 0)
+			(effects
+				(font
+					(size 1.27 1.27)
+				)
+				(justify left)
+			)
+		)
+		(property "Footprint" "Swadge_Parts:C_Radial_D4_L5.4_P3.321"
+			(at 166.37 193.04 0)
+			(effects
+				(font
+					(size 1.27 1.27)
+				)
+				(hide yes)
+			)
+		)
+		(property "Datasheet" "~"
+			(at 166.37 193.04 0)
+			(effects
+				(font
+					(size 1.27 1.27)
+				)
+				(hide yes)
+			)
+		)
+		(property "Description" "Polarized capacitor, US symbol"
+			(at 166.37 193.04 0)
+			(effects
+				(font
+					(size 1.27 1.27)
+				)
+				(hide yes)
+			)
+		)
+		(property "Digikey" "~"
+			(at 169.545 187.96 0)
+			(effects
+				(font
+					(size 1.27 1.27)
+				)
+				(hide yes)
+			)
+		)
+		(property "Cost100" "510"
+			(at 166.37 193.04 0)
+			(effects
+				(font
+					(size 0.254 0.254)
+				)
+				(hide yes)
+			)
+		)
+		(property "Substitutable" "Y"
+			(at 166.37 193.04 0)
+			(effects
+				(font
+					(size 0.001 0.001)
+				)
+				(hide yes)
+			)
+		)
+		(property "LCSC" "C2895732"
+			(at 166.37 193.04 0)
+			(effects
+				(font
+					(size 1.27 1.27)
+				)
+				(hide yes)
+			)
+		)
+		(property "Cost @ 2.5k" "0.0147"
+			(at 166.37 193.04 0)
+			(effects
+				(font
+					(size 1.27 1.27)
+				)
+				(hide yes)
+			)
+		)
+		(pin "1"
+		)
+		(pin "2"
+		)
+		(instances
+			(project "Swadge-HW"
+				(path "/770c762f-3a30-4864-b7da-de353459cdd6"
+					(reference "C26")
+					(unit 1)
+				)

Commit message: Generate RB manufacturing data, small edits
Change footprint for C26 + BOM Data
Add notch in Acrylic for fitment
Update schematic to reflect C26 change
Add quote data
Update condiment dxf/svg
Parts:
- C26: Cost @ 2.5k 0.0147 -> 0.031; Cost100 510 -> 31; LCSC C2895732 -> C7465562
Changed lines of the file:
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@@
 			)
 		)
-		(property "Cost100" "510"
+		(property "Cost100" "31"
 			(at 166.37 193.04 0)
 			(effects
@@
 			)
 		)
-		(property "LCSC" "C2895732"
+		(property "LCSC" "C7465562"
 			(at 166.37 193.04 0)
 			(effects
@@
 			)
 		)
-		(property "Cost @ 2.5k" "0.0147"
+		(property "Cost @ 2.5k" "0.031"
 			(at 166.37 193.04 0)
 			(effects

Commit message: Update mfg files
Updated mfg files for elecrow quote
Parts:
- C21: LCSC C282519 -> C6119848
Changed lines of the file:
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@@
 			)
 		)
-		(property "LCSC" "C282519"
+		(property "LCSC" "C6119848"
 			(at 261.62 134.62 0)
 			(effects
